File: BreakBeamEmitter.brd (EAGLE design)
At the start: 53.3 x 35.6 mm, 11 parts, among them IC1 LM555N

Commit message: Updates
Parts:
- R4: value 2.2K -> 1K
Changed lines of the file:
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@@
 <element name="R1" library="SparkFun-Resistors" package="AXIAL-0.3" value="10K" x="24.13" y="20.32"/>
 <element name="R3" library="SparkFun-Resistors" package="AXIAL-0.3" value="27K" x="24.13" y="25.4" rot="R180"/>
-<element name="R4" library="SparkFun-Resistors" package="AXIAL-0.3" value="2.2K" x="24.13" y="22.86"/>
+<element name="R4" library="SparkFun-Resistors" package="AXIAL-0.3" value="1K" x="24.13" y="22.86"/>
 <element name="R6" library="resistor" package="RTRIM64Y" value="5K" x="33.02" y="25.4"/>
 <element name="C2" library="SparkFun-Capacitors" package="CAP-PTH-5MM" value="10nF" x="33.02" y="15.24" rot="R90"/>
@@
 <wire x1="12.7" y1="12.7" x2="12.7" y2="12.74" width="0.4064" layer="16"/>
 </signal>
-<signal name="N$1">
-<contactref element="IC1" pad="7"/>
-<contactref element="R1" pad="P$2"/>
-<contactref element="R4" pad="P$2"/>
-<wire x1="27.94" y1="22.86" x2="27.94" y2="20.32" width="0.4064" layer="16"/>
-<wire x1="27.94" y1="20.32" x2="25.4" y2="17.78" width="0.4064" layer="16"/>
-</signal>
 <signal name="N$2">
 <contactref element="IC1" pad="6"/>
@@
 <wire x1="27.94" y1="10.16" x2="27.94" y2="7.62" width="0.4064" layer="16"/>
 </signal>
+<signal name="N$8">
+<contactref element="IC1" pad="7"/>
+<contactref element="R1" pad="P$2"/>
+<wire x1="27.94" y1="20.32" x2="25.4" y2="17.78" width="0.4064" layer="16"/>
+<contactref element="R4" pad="P$2"/>
+<wire x1="27.94" y1="20.32" x2="27.94" y2="22.86" width="0.4064" layer="16"/>
+</signal>
 </signals>
