File: BreakBeamEmitter.sch (EAGLE design)
At the start: 11 parts, among them IC1 LM555N

Commit message: Updates
Parts:
- R4: value 2.2K -> 1K
Other:
- moved on the sheet: C3
Changed lines of the file:
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@@
 <part name="P+4" library="supply1" deviceset="VCC" device=""/>
 <part name="R3" library="SparkFun-Resistors" deviceset="RESISTOR" device="AXIAL-0.3" value="27K"/>
-<part name="R4" library="SparkFun-Resistors" deviceset="RESISTOR" device="AXIAL-0.3" value="2.2K"/>
+<part name="R4" library="SparkFun-Resistors" deviceset="RESISTOR" device="AXIAL-0.3" value="1K"/>
 <part name="R6" library="resistor" deviceset="R-TRIMM" device="64Y" value="5K"/>
 <part name="C2" library="SparkFun-Capacitors" deviceset="CAP" device="PTH1" value="10nF"/>
@@
 <instance part="LED1" gate="G$1" x="71.12" y="78.74" rot="R180"/>
 <instance part="P+5" gate="VCC" x="71.12" y="86.36"/>
-<instance part="GND4" gate="1" x="78.74" y="30.48"/>
-<instance part="C3" gate="G$1" x="78.74" y="38.1" rot="R180"/>
+<instance part="GND4" gate="1" x="78.74" y="27.94"/>
+<instance part="C3" gate="G$1" x="78.74" y="35.56" rot="R180"/>
 </instances>
 <busses>
@@
 </segment>
 </net>
-<net name="N$1" class="0">
-<segment>
-<pinref part="IC1" gate="A" pin="DIS"/>
-<pinref part="R1" gate="G$1" pin="2"/>
-<wire x1="83.82" y1="50.8" x2="71.12" y2="50.8" width="0.1524" layer="91"/>
-<wire x1="83.82" y1="50.8" x2="83.82" y2="55.88" width="0.1524" layer="91"/>
-<junction x="83.82" y="50.8"/>
-<wire x1="83.82" y1="55.88" x2="104.14" y2="55.88" width="0.1524" layer="91"/>
-<pinref part="R4" gate="G$1" pin="2"/>
-<wire x1="104.14" y1="55.88" x2="104.14" y2="35.56" width="0.1524" layer="91"/>
-</segment>
-</net>
 <net name="N$2" class="0">
 <segment>
@@
 <junction x="73.66" y="45.72"/>
 <pinref part="R6" gate="G$1" pin="E"/>
-<wire x1="78.74" y1="45.72" x2="78.74" y2="40.64" width="0.1524" layer="91"/>
+<wire x1="78.74" y1="45.72" x2="78.74" y2="38.1" width="0.1524" layer="91"/>
 <pinref part="C3" gate="G$1" pin="2"/>
-<junction x="78.74" y="40.64"/>
+<junction x="78.74" y="38.1"/>
+<wire x1="78.74" y1="38.1" x2="78.74" y2="40.64" width="0.1524" layer="91"/>
 </segment>
 </net>
@@
 </segment>
 </net>
+<net name="N$8" class="0">
+<segment>
+<pinref part="IC1" gate="A" pin="DIS"/>
+<pinref part="R1" gate="G$1" pin="2"/>
+<wire x1="83.82" y1="50.8" x2="71.12" y2="50.8" width="0.1524" layer="91"/>
+<wire x1="83.82" y1="50.8" x2="83.82" y2="45.72" width="0.1524" layer="91"/>
+<junction x="83.82" y="50.8"/>
+<wire x1="83.82" y1="45.72" x2="104.14" y2="45.72" width="0.1524" layer="91"/>
+<pinref part="R4" gate="G$1" pin="2"/>
+<wire x1="104.14" y1="45.72" x2="104.14" y2="35.56" width="0.1524" layer="91"/>
+</segment>
+</net>
